Commit message: feat: add RoboTest showcase presentation

File: src/robotest_description/urdf/robotest_base.xacro (robot description, xacro)
@@ -7,5 +7,5 @@
   <xacro:macro name="robotest_wheel" params="side y">
     <link name="${side}_wheel_link">
-      <visual>
+      <visual name="${side}_wheel_tire_visual">
         <origin xyz="0 0 0" rpy="${pi / 2.0} 0 0"/>
         <geometry>
@@ -13,4 +13,18 @@
         </geometry>
         <material name="robotest_dark"/>
+      </visual>
+      <visual name="${side}_wheel_rim_visual">
+        <origin xyz="0 0 0" rpy="${pi / 2.0} 0 0"/>
+        <geometry>
+          <cylinder radius="${wheel_radius * 0.55}" length="${wheel_width + 0.006}"/>
+        </geometry>
+        <material name="robotest_silver"/>
+      </visual>
+      <visual name="${side}_wheel_hub_visual">
+        <origin xyz="0 0 0" rpy="${pi / 2.0} 0 0"/>
+        <geometry>
+          <cylinder radius="${wheel_radius * 0.22}" length="${wheel_width + 0.012}"/>
+        </geometry>
+        <material name="robotest_sensor"/>
       </visual>
       <collision name="${side}_wheel_collision">
@@ -58,9 +72,54 @@
     <link name="base_footprint"/>
     <link name="base_link">
-      <visual>
+      <!-- Presentation geometry is deliberately separate from the frozen
+           collision and inertial envelopes below. -->
+      <visual name="lower_chassis_visual">
+        <origin xyz="0 0 -0.015" rpy="0 0 0"/>
         <geometry>
-          <box size="${base_length} ${base_width} ${base_height}"/>
+          <box size="${base_length} ${base_width} 0.09"/>
+        </geometry>
+        <material name="robotest_navy"/>
+      </visual>
+      <visual name="upper_chassis_visual">
+        <origin xyz="-0.015 0 0.06" rpy="0 0 0"/>
+        <geometry>
+          <box size="0.39 0.27 0.085"/>
         </geometry>
         <material name="robotest_blue"/>
+      </visual>
+      <visual name="top_deck_visual">
+        <origin xyz="-0.005 0 0.1125" rpy="0 0 0"/>
+        <geometry>
+          <box size="0.32 0.23 0.02"/>
+        </geometry>
+        <material name="robotest_silver"/>
+      </visual>
+      <visual name="front_bumper_visual">
+        <origin xyz="0.245 0 -0.0125" rpy="0 0 0"/>
+        <geometry>
+          <box size="0.03 0.34 0.055"/>
+        </geometry>
+        <material name="robotest_sensor"/>
+      </visual>
+      <visual name="left_headlight_visual">
+        <origin xyz="0.262 0.09 0.035" rpy="0 0 0"/>
+        <geometry>
+          <sphere radius="0.024"/>
+        </geometry>
+        <material name="robotest_light"/>
+      </visual>
+      <visual name="right_headlight_visual">
+        <origin xyz="0.262 -0.09 0.035" rpy="0 0 0"/>
+        <geometry>
+          <sphere radius="0.024"/>
+        </geometry>
+        <material name="robotest_light"/>
+      </visual>
+      <visual name="lidar_mast_visual">
+        <origin xyz="${lidar_x} 0 0.095" rpy="0 0 0"/>
+        <geometry>
+          <cylinder radius="0.047" length="0.07"/>
+        </geometry>
+        <material name="robotest_navy"/>
       </visual>
       <collision name="base_link_collision">

File: src/robotest_description/urdf/robotest_materials.xacro (robot description, xacro)
@@ -14,3 +14,12 @@
     <color rgba="0.94 0.48 0.10 1.0"/>
   </material>
+  <material name="robotest_navy">
+    <color rgba="0.03 0.08 0.18 1.0"/>
+  </material>
+  <material name="robotest_silver">
+    <color rgba="0.62 0.68 0.76 1.0"/>
+  </material>
+  <material name="robotest_light">
+    <color rgba="0.86 0.95 1.0 1.0"/>
+  </material>
 </robot>

File: src/robotest_description/urdf/robotest_sensors.xacro (robot description, xacro)
@@ -7,9 +7,24 @@
   <xacro:macro name="robotest_sensors">
     <link name="lidar_link">
-      <visual>
+      <visual name="lidar_lower_housing_visual">
+        <origin xyz="0 0 -0.005" rpy="0 0 0"/>
         <geometry>
-          <cylinder radius="${lidar_radius}" length="${lidar_height}"/>
+          <cylinder radius="${lidar_radius + 0.012}" length="0.035"/>
+        </geometry>
+        <material name="robotest_navy"/>
+      </visual>
+      <visual name="lidar_scan_head_visual">
+        <origin xyz="0 0 0.0225" rpy="0 0 0"/>
+        <geometry>
+          <cylinder radius="${lidar_radius + 0.004}" length="0.032"/>
         </geometry>
         <material name="robotest_sensor"/>
+      </visual>
+      <visual name="lidar_top_cap_visual">
+        <origin xyz="0 0 0.041" rpy="0 0 0"/>
+        <geometry>
+          <cylinder radius="${lidar_radius * 0.72}" length="0.008"/>
+        </geometry>
+        <material name="robotest_silver"/>
       </visual>
       <collision name="lidar_link_collision">
